File: Petoi/Electronics/RRLInterface/rrl-interface.sch (KiCad schematic (older format))
At the start: 14 parts, among them J1 Legs, J2 USB pwr out, J3 I2C, J4 range, U1 LTC2990

Commit message: Sally's latest design for the leg PCB.
Parts:
- added C4: 1u, Capacitor_SMD:C_0805_2012Metric, symbol Device:C
Connections:
- net at D1.1 (+), D2.1 (+), J2.2 (Pin_2): now also C4.2
- net at D1.2 (-), D2.2 (-), J2.1 (Pin_1): now also C4.1
Changed lines of the file:
@@
 $EndComp
 Wire Wire Line
-	2850 1250 2300 1250
+	2850 1250 2500 1250
 Connection ~ 2300 1250
 Wire Wire Line
 	2300 1250 2300 1800
 Wire Wire Line
-	2850 1350 1450 1350
+	2850 1350 2800 1350
 Connection ~ 1450 1350
 Wire Wire Line
@@
 	6100 1275 6225 1275
 Connection ~ 5975 1475
+$Comp
+L Device:C C4
+U 1 1 627BBE63
+P 2650 1500
+F 0 "C4" H 2765 1546 50  0000 L CNN
+F 1 "1u" H 2765 1455 50  0000 L CNN
+F 2 "Capacitor_SMD:C_0805_2012Metric" H 2688 1350 50  0001 C CNN
+F 3 "~" H 2650 1500 50  0001 C CNN
+	1    2650 1500
+	0    1    1    0
+$EndComp
+Wire Wire Line
+	2800 1500 2800 1350
+Connection ~ 2800 1350
+Wire Wire Line
+	2800 1350 1450 1350
+Wire Wire Line
+	2500 1500 2500 1250
+Connection ~ 2500 1250
+Wire Wire Line
+	2500 1250 2300 1250
 $EndSCHEMATC

Commit message: Sally improved PCB
Parts:
- removed C2, C3: 0.1u, Capacitor_SMD:C_0805_2012Metric, symbol Device:C
- added C5, C6, C8: 0.1u, Capacitor_SMD:C_0805_2012Metric, symbol Device:C
- added J5, J7: I2C, Connector_PinSocket_2.54mm:PinSocket_1x04_P2.54mm_Vertical, symbol Connector:Conn_01x04_Male
- added J6, J8: range, Connector_PinSocket_2.54mm:PinSocket_1x04_P2.54mm_Vertical, symbol Connector:Conn_01x04_Male
Connections:
- net +3V3: now also C5.1, C6.1, C8.1, J5.1 (Pin_1), J6.1 (Pin_1), J7.1 (Pin_1), J8.1 (Pin_1)
- net GND: now also C5.2, C6.2, C8.2, J5.2 (Pin_2), J6.2 (Pin_2), J7.2 (Pin_2), J8.2 (Pin_2)
- net SCL: now also J5.4 (Pin_4), J6.4 (Pin_4), J7.4 (Pin_4), J8.4 (Pin_4)
- net SDA: now also J5.3 (Pin_3), J6.3 (Pin_3), J7.3 (Pin_3), J8.3 (Pin_3)

Commit message: Updating electronics
Parts:
- J4, J8: value range -> I2C
- J7: value I2C -> OLED
Other:
- moved on the sheet: C5, C6, C8, J4, J5, J6, J7, J8
