File: Petoi/Electronics/RRLInterface/rrl-interface.kicad_pcb (KiCad board)
At the start: 2 copper layers, 26 x 65 mm, 14 parts, among them J1 Legs, J2 USB pwr out, J3 I2C, J4 range, U1 LTC2990

Commit message: Sally's latest design for the leg PCB.
Parts:
- added C4: 1u, Capacitor_SMD:C_0805_2012Metric, B.Cu at (23.4, 189.3)
- moved H3 255.5 mm to (74.5, 192.5), turned to 270 degrees
- moved J3 248.5 mm to (73.5, 186.9), turned to 180 degrees
- moved C3 248.1 mm to (64.8, 182.6), turned to 0 degrees
- moved J1 245.5 mm to (66.7, 192.5), turned to 270 degrees
- moved J4 245.4 mm to (70.0, 186.9), turned to 180 degrees
- moved C1 241.5 mm to (67.0, 185.7), turned to 90 degrees
- moved C2 237.4 mm to (76.6, 185.8)
- moved H2 235.2 mm to (74.5, 173.5), turned to 270 degrees
- moved U1 230.4 mm to (63.6, 179.4), turned to 0 degrees
- moved H4 214.0 mm to (16.5, 192.5), turned to 270 degrees
- moved J2 213.0 mm to (22.1, 192.5)
- moved D1 207.2 mm to (56.5, 181.5), turned to 270 degrees
- moved D2 198.4 mm to (46.4, 181.6), turned to 270 degrees
- moved H1 189.3 mm to (16.5, 173.5), turned to 270 degrees
Routing:
- net GND: track 75.6 -> 5.31 mm, vias 6 -> 0
- net Net-(J1-Pad16): track 70.5 -> 45.2 mm
- net Net-(C4-Pad1): track 17.6 -> 40.1 mm
- net Net-(D2-Pad4): track 20.7 -> 3.32 mm
- net Net-(D1-Pad4): track 28.9 -> 11.6 mm, vias 2 -> 0
- net +3V3: track 84.8 -> 70.8 mm
- net Net-(D1-Pad3): track 19.0 -> 6.54 mm, vias 2 -> 0
- net Net-(C4-Pad2): track 30.9 -> 42.2 mm
- net Net-(J1-Pad4): track 17.9 -> 13.5 mm
- net Net-(D2-Pad3): track 10.8 -> 6.46 mm
- net SCL: track 12.1 -> 7.87 mm
- net SDA: track 23.6 -> 22.0 mm
- net Net-(J1-Pad12): track 35.8 -> 36.2 mm, vias 2 -> 0
- added copper zone on F.Cu, net GND
Other:
- board size 26 x 65 mm -> 65 x 26 mm
- board text added: "Petoi Robot Legs Interface RepRap Ltd https://reprapltd.com Licence: GPL Version 1 Design: Sally Bowyer"

Commit message: Keeping things up to date
Parts:
- ?: renamed from H4; value MountingHole -> (none)
- ?: renamed from J1; value Legs -> (none)
- ?: renamed from U1; value LTC2990 -> (none)
- ?: renamed from J2; value USB pwr out -> (none)
- ?: renamed from H1; value MountingHole -> (none)
- ?: renamed from H2; value MountingHole -> (none)
- ?: renamed from H3; value MountingHole -> (none)
- renumbered D1 to ?, J3 to ?, J4 to ?, C4 to ?, D2 to ?, C1 to ?, C2 to ?, C3 to ?
Routing:
- net Net-(D1-Pad4): track 11.6 -> 12.7 mm
Other:
- board text added: "+"
- board text added: "-"
- board text added: "3V3"
- board text added: "DF06M"
- board text added: "F"
- board text added: "G"
- board text added: "GND"
- board text added: "I2C"
- board text added: "LTC2990"
- board text added: "P"
- board text added: "SCL"
- board text added: "SDA"
- board text added: "legs"
- board text added: "pwr out"
- board text added: "range"

Commit message: Sally improved PCB
Parts:
- removed ?: I2C, Connector_PinSocket_2.54mm:PinSocket_1x04_P2.54mm_Vertical
- removed ?: range, Connector_PinSocket_2.54mm:PinSocket_1x04_P2.54mm_Vertical
- removed ? (x2): 0.1u, Capacitor_SMD:C_0805_2012Metric
- added C5: 0.1u, Capacitor_SMD:C_0805_2012Metric, B.Cu at (57.8, 185.2)
- added C6: 0.1u, Capacitor_SMD:C_0805_2012Metric, B.Cu at (67.6, 185.2)
- added C8: 0.1u, Capacitor_SMD:C_0805_2012Metric, B.Cu at (48.0, 185.2)
- added J3: I2C, Connector_PinSocket_2.54mm:PinSocket_1x04_P2.54mm_Vertical, F.Cu at (54.8, 186.8)
- added J4: range, Connector_PinSocket_2.54mm:PinSocket_1x04_P2.54mm_Vertical, F.Cu at (51.0, 186.8)
- added J5: I2C, Connector_PinSocket_2.54mm:PinSocket_1x04_P2.54mm_Vertical, F.Cu at (74.4, 186.8)
- added J6: range, Connector_PinSocket_2.54mm:PinSocket_1x04_P2.54mm_Vertical, F.Cu at (70.6, 186.8)
- added J7: I2C, Connector_PinSocket_2.54mm:PinSocket_1x04_P2.54mm_Vertical, F.Cu at (64.6, 186.8)
- added J8: range, Connector_PinSocket_2.54mm:PinSocket_1x04_P2.54mm_Vertical, F.Cu at (60.8, 186.8)
- H1, H2, H3, H4: renamed from ?; value (none) -> MountingHole
- J1: renamed from ?; value (none) -> Legs
- J2: renamed from ?; value (none) -> USB pwr out
- U1: renamed from ?; value (none) -> LTC2990
- moved C1 19.4 mm to (48.0, 181.6), turned to 270 degrees
- moved U1 18.3 mm to (45.8, 175.0)
- moved D1 16.7 mm to (40.0, 179.0)
- moved D2 16.6 mm to (30.0, 179.0)
- moved J2 12.6 mm to (16.0, 181.4), turned to 180 degrees
- moved C4 10.1 mm to (19.0, 180.2), turned to 90 degrees
- moved J1 6.76 mm to (59.9, 192.6)
- gave numbers to parts that had none: 4
Routing:
- net SCL: track 7.87 -> 30.4 mm
- net Net-(C4-Pad1): track 40.1 -> 21.4 mm
- net Net-(C4-Pad2): track 42.2 -> 26.4 mm
- net SDA: track 22.0 -> 36.7 mm
- net +3V3: track 70.8 -> 85.4 mm
- net Net-(J1-Pad12): track 36.2 -> 23.6 mm
- net Net-(D1-Pad3): track 6.72 -> 18.1 mm
- net Net-(J1-Pad4): track 13.5 -> 23.8 mm
- net Net-(D2-Pad4): track 3.32 -> 13.1 mm
- net Net-(D1-Pad4): track 12.7 -> 22.4 mm
- net Net-(J1-Pad16): track 45.2 -> 53.2 mm
- net Net-(J1-Pad8): track 23.7 -> 19.0 mm
- net Net-(D2-Pad3): track 6.46 -> 11.0 mm

Commit message: Updating electronics
Parts:
- J4, J8: value range -> I2C
- J7: value I2C -> OLED
- moved C4 3.94 mm to (20.6, 183.8)
- moved J2 3.41 mm to (16.2, 184.8)
Routing:
- net Net-(C4-Pad2): track 26.4 -> 35.8 mm
- net Net-(C4-Pad1): track 21.4 -> 27.3 mm
- net +3V3: track 85.4 -> 87.0 mm
- net Net-(D1-Pad4): track 22.4 -> 23.5 mm
- net Net-(D2-Pad3): track 11.0 -> 11.7 mm
Other:
- board text added: "Licence: GPL Version: 2 Design: Sally Bowyer"
- board text added: "Petoi Robot Legs Interface RepRap Ltd https://reprapltd.com"
- board text removed: "DF06M"
- board text removed: "Petoi Robot Legs Interface RepRap Ltd https://reprapltd.com Licence: GPL Version 1 Design: Sally Bowyer"
- board text removed: "range"

Commit message: Starting work* on a graphical simulator for the Petoi robot.
* GPT4 doing the heavy lifting. Life is short...
Other:
- net class Default removed
